File: PCB_Designs/Basic/WalkieTalkie_Basic.brd (EAGLE design)
At the start: 33 x 50.8 mm, 60 parts, among them IC1 AD8609RU, IC2 AD8603UJ, IC3 MCP601OT, Q1 MOSFET-NCHANNELBSS123LT1G

Commit message: more updates to PCB almost done
Parts:
- moved R2 7.34 mm to (27.7, 22.1), turned to 90 degrees
- moved R3 5.35 mm to (23.9, 16.7), turned to 270 degrees
- moved R1 5.24 mm to (27.7, 19.5), turned to 90 degrees
- moved C20 4.91 mm to (23.0, 20.2), turned to 270 degrees
- moved Q1 4.20 mm to (25.5, 19.9)
- moved C9 4.17 mm to (7.06, 37.1), turned to 180 degrees
- moved C1 2.56 mm to (25.7, 17.3), turned to 180 degrees
- moved XTAL 1.37 mm to (19.7, 26.4), turned to 270 degrees
- moved C14 1.19 mm to (21.7, 24.8), turned to 180 degrees
- moved R6 0.72 mm to (9.30, 23.8), turned to 90 degrees
- moved C22 0.62 mm to (12.0, 21.3)
- moved C15 0.31 mm to (21.7, 26.2), turned to 180 degrees
Connections:
- new net N$22: ARDUINO.25
- new net N$25: ARDUINO.26
- new net N$29: ARDUINO.27
- new net N$30: ARDUINO.28
- new net N$31: ARDUINO.19
- new net N$32: ARDUINO.22
Routing:
- net A0-MIC: track 0.00 -> 27.5 mm, vias 0 -> 3
- net 3.3V: track 1.03 -> 17.6 mm, vias 1 -> 10
- net GND: track 2.76 -> 17.5 mm, vias 1 -> 6
- net D3: track 15.3 -> 21.5 mm, vias 0 -> 1
- net N$2: track 0.00 -> 5.49 mm, vias 0 -> 1
- net N$8: track 0.00 -> 3.32 mm
- net N$21: track 5.64 -> 2.67 mm
- net N$5: track 0.00 -> 2.85 mm
- net N$20: track 6.82 -> 4.61 mm
- net D6: track 14.4 -> 13.0 mm

Commit message: more updates almost done
Parts:
- added S1: TAC_SWITCHSMD, SparkFun-Retired:TACTILE-SWITCH-SMD
- moved LDO 24.6 mm to (27.6, 17.1), turned to 0 degrees
- moved C24 22.3 mm to (25.7, 17.1), turned to 270 degrees
- moved LIPO 21.5 mm to (30.5, 17.4), turned to 270 degrees
- moved C23 20.5 mm to (29.1, 14.7), turned to 270 degrees
- moved R18 2.01 mm to (6.91, 28.9), turned to 180 degrees
- moved R16 1.62 mm to (17.3, 31.7), turned to 270 degrees
- moved C4 1.35 mm to (16.6, 37.2), turned to 180 degrees
- moved C17 0.95 mm to (16.1, 36.5)
- moved C14 0.95 mm to (21.3, 25.7), flipped to the bottom, turned to 0 degrees
- moved C15 0.84 mm to (21.3, 26.9), flipped to the bottom, turned to 0 degrees
- moved R11 0.64 mm to (8.59, 24.0)
- moved R6 0.55 mm to (9.80, 24.0)
- moved XTAL 0.51 mm to (19.7, 26.9)
- moved R17 0.20 mm to (4.47, 26.5)
- moved CALL 0.20 mm to (13.2, 16.1)
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Connections:
- new net N$34: CALL.3
- net GND: now also CALL.4, TALK.4; no longer CALL.2, TALK.2
- net N$1: now also TALK.2; no longer C21.2, CALL.1, R21.2
- net N$2: now also TALK.3; no longer C2.2, R4.2, TALK.1
- net TALK/CALL: now also C2.2, C21.2, CALL.1, R21.2, R4.2, TALK.1; no longer CALL.4, TALK.4
Routing:
- net V_BATT: track 0.00 -> 7.08 mm
- net GND: track 17.5 -> 23.7 mm, vias 6 -> 8
- net N$2: track 5.49 -> 0.00 mm, vias 1 -> 0
- net N$3: track 18.4 -> 14.3 mm
- net N$1: track 4.11 -> 0.00 mm, vias 1 -> 0
- net D2-IRQ: track 30.2 -> 27.3 mm
- net N$24: track 7.21 -> 4.88 mm
- net N$28: track 0.00 -> 1.29 mm
- net D11-MOSI: track 26.5 -> 25.4 mm
- net TALK/CALL: track 25.1 -> 26.2 mm, vias 2 -> 4
- net N$20: track 4.61 -> 3.86 mm
- net N$23: track 2.64 -> 1.97 mm
- net D3: track 21.5 -> 20.9 mm
- net RESET: track 14.8 -> 15.4 mm
