File: PCB_Designs/Basic/WalkieTalkie_Basic.sch (EAGLE design)
At the start: 61 parts, among them IC1 AD8609RU, IC2 AD8603UJ, IC3 MCP601OT, Q1 MOSFET-NCHANNELBSS123LT1G

Commit message: updates. almost done
Parts:
- added U$4: PS1240P02CT3P, Orlando:PS1240P02CT3P
Connections:
- net GND: now also LIPO-.TP; no longer LIPOG$1.TP
- net V_BATT: now also LIPO+.TP; no longer LIPOG$2.TP
Changed lines of the file:
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@@
 <?xml version="1.0" encoding="utf-8"?>
 <!DOCTYPE eagle SYSTEM "eagle.dtd">
-<eagle version="7.4.0">
+<eagle version="7.3.0">
 <drawing>
 <settings>
@@
 <part name="GND16" library="SparkFun-Aesthetics" deviceset="GND" device=""/>
 <part name="S1" library="SparkFun-Retired" deviceset="TAC_SWITCH" device="SMD" value="TAC_SWITCHSMD"/>
+<part name="U$4" library="Orlando" deviceset="PS1240P02CT3" device="P"/>
 </parts>
 <sheets>
@@
 <instance part="LDO" gate="G$1" x="228.6" y="71.12"/>
 <instance part="GND25" gate="1" x="213.36" y="58.42"/>
-<instance part="LIPO" gate="G$2" x="182.88" y="63.5"/>
-<instance part="LIPO" gate="G$1" x="190.5" y="63.5"/>
+<instance part="LIPO" gate="-" x="190.5" y="63.5"/>
+<instance part="LIPO" gate="+" x="182.88" y="63.5"/>
 <instance part="GND26" gate="1" x="195.58" y="63.5"/>
 <instance part="SUPPLY13" gate="G$1" x="182.88" y="81.28"/>
@@
 <instance part="GND16" gate="1" x="-20.32" y="53.34"/>
 <instance part="S1" gate="S" x="116.84" y="106.68"/>
+<instance part="U$4" gate="G$1" x="170.18" y="27.94"/>
 </instances>
 <busses>
@@
 </segment>
 <segment>
-<pinref part="LIPO" gate="G$1" pin="TP"/>
-<wire x1="190.5" y1="66.04" x2="190.5" y2="68.58" width="0.1524" layer="91"/>
 <wire x1="190.5" y1="68.58" x2="195.58" y2="68.58" width="0.1524" layer="91"/>
 <wire x1="195.58" y1="68.58" x2="195.58" y2="66.04" width="0.1524" layer="91"/>
 <pinref part="GND26" gate="1" pin="GND"/>
+<pinref part="LIPO" gate="-" pin="TP"/>
+<wire x1="190.5" y1="66.04" x2="190.5" y2="68.58" width="0.1524" layer="91"/>
 </segment>
 <segment>
@@
 <net name="V_BATT" class="0">
 <segment>
-<pinref part="LIPO" gate="G$2" pin="TP"/>
-<wire x1="182.88" y1="66.04" x2="182.88" y2="76.2" width="0.1524" layer="91"/>
 <pinref part="SUPPLY13" gate="G$1" pin="V_BATT"/>
 <pinref part="LDO" gate="G$1" pin="IN"/>
@@
 <junction x="215.9" y="76.2"/>
 <wire x1="205.74" y1="76.2" x2="182.88" y2="76.2" width="0.1524" layer="91"/>
+<pinref part="LIPO" gate="+" pin="TP"/>
+<wire x1="182.88" y1="66.04" x2="182.88" y2="76.2" width="0.1524" layer="91"/>
 <junction x="182.88" y="76.2"/>
 </segment>

Commit message: finished board design. sent to fab (OSH Park)
Parts:
- removed S1: TAC_SWITCHSMD, SparkFun-Retired:TAC_SWITCHSMD
- removed U$4: PS1240P02CT3P, Orlando:PS1240P02CT3P
- renumbered IC1 to AUDIO, IC2 to VREF, PROGRAM/BOOTLOAD to PROGRAM/BOOTLOADING, Q1 to MIC-AMP, U$3 to NRF24

Commit message: updated pcb files with comments, labels, etc
Parts:
- added LOGO1: OSHW-LOGOS, SparkFun-Aesthetics:OSHW-LOGOS
- renumbered D2 to NOTIFY
Connections:
- net D3: no longer U$2.+
- net D5: now also U$2.+
Other:
- note added: "Bootloading/ Programming"
- note added: "Call Notification"
- note added: "Call and Talk Buttons"
- note added: "Maybe a switch to turn it off, or a potentiometer to turn the volume down some button to switch channels and LEDs to indicate what channel we're on"
- note added: "Mircophone Pre-amp"
- note added: "Regulator"
- note added: "Sound Out and Filtering Circuit"
- note added: "nRF24L01"
- note removed: "LED to indicate when the device is powered Maybe a switch to turn it off, or a potentiometer to turn the volume down LED to indicate when a call has been received LED to indicate when a call is being made LED to indicate when two devices are talking some button to switch channels and LEDs to indicate what channel we're on"
- note removed: "Some sort of volume control"
- moved on the sheet: AUDIOA, AUDIOB, AUDIOC, AUDIOD, AUDIOP, C1, C10, C11, C12, C13, C18, C19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
